Commit message: Hardware Interface working

File: test/description/gazebo_control.xacro (robot description, xacro)
@@ -5,6 +5,6 @@
             <left_joint>left_wheel_joint</left_joint>
             <right_joint>right_wheel_joint</right_joint>
-            <wheel_separation>0.35</wheel_separation>
-            <wheel_diameter>0.1</wheel_diameter>
+            <wheel_separation>0.18</wheel_separation>
+            <wheel_diameter>0.66</wheel_diameter>
             <max_wheel_torque>200</max_wheel_torque>
             <max_wheel_acceleration>10.0</max_wheel_acceleration>

File: test/description/robot.urdf.xacro (robot description, xacro)
@@ -2,5 +2,6 @@
 <robot xmlns:xacro="http://www.ros.org/wiki/xacro" name="robot_jet">
 <xacro:include filename="robot_core.xacro"/>
-<xacro:include filename="gazebo_control.xacro"/>
+<!-- <xacro:include filename="gazebo_control.xacro"/> -->
 <xacro:include filename="camera.xacro"/>
+<xacro:include filename="diffbot.urdf.xacro"/>
 </robot>

File: test/description/robot_core.xacro (robot description, xacro)
@@ -22,22 +22,22 @@
     <parent link="base_link"/>
     <child link="chassis"/>
-    <origin xyz="-0.1 0.0 0.0"/>
+    <origin xyz="-0.015 0.0 0.00"/>
 </joint>
 <link name="chassis">
     <visual>
-    <origin xyz="0.15 0.0 0.075"/>
+    <origin xyz="0.059 0.0 0.0225"/>
         <geometry>
-            <box size="0.3 0.3 0.15"/>
+            <box size="0.118 0.167 0.045"/>
         </geometry>
         <material name="white"/>
     </visual>
     <collision>
-        <origin xyz="0.15 0.0 0.075"/>
+        <origin xyz="0.059 0.0 0.0225"/>
         <geometry>
-            <box size="0.3 0.3 0.15"/>
+            <box size="0.118 0.167 0.045"/>
         </geometry>
     </collision>
-    <xacro:inertial_box mass="0.3" x="0.3" y="0.3" z="0.15">
-        <origin xyz="0.15 0.0 0.075" rpy="0.0 0.0 0.0"/>
+    <xacro:inertial_box mass="0.3" x="0.118" y="0.167" z="0.045">
+        <origin xyz="0.059 0.0 0.0225" rpy="0.0 0.0 0.0"/>
     </xacro:inertial_box>
     <gazebo reference="chassis">
@@ -49,5 +49,5 @@
     <parent link="base_link"/>
     <child link="left_wheel"/>
-    <origin xyz="0.0 0.175 0.0" rpy="-${pi/2} 0.0 0.0"/>
+    <origin xyz="0.0 0.090 0.0" rpy="-${pi/2} 0.0 0.0"/>
     <axis xyz="0.0 0.0 1.0"/>
 </joint>
@@ -58,5 +58,5 @@
     <visual>
         <geometry>
-            <cylinder radius="0.05" length="0.04"/>
+            <cylinder radius="0.033" length="0.022"/>
         </geometry>
         <material name="blue"/>
@@ -64,8 +64,8 @@
     <collision>
         <geometry>
-            <cylinder radius="0.05" length="0.04"/>
+            <cylinder radius="0.033" length="0.022"/>
         </geometry>
     </collision>
-    <xacro:inertial_cylinder mass="0.1" length="0.04" radius="0.05">
+    <xacro:inertial_cylinder mass="0.1" radius="0.033" length="0.022">
         <origin xyz="0.0 0.0 0.0" rpy="0.0 0.0 0.0"/>
     </xacro:inertial_cylinder>
@@ -78,5 +78,5 @@
     <parent link="base_link"/>
     <child link="right_wheel"/>
-    <origin xyz="0.0 -0.175 0.0" rpy="${pi/2} 0.0 0.0"/>
+    <origin xyz="0.0 -0.090 0.0" rpy="${pi/2} 0.0 0.0"/>
     <axis xyz="0.0 0.0 -1.0"/>
 </joint>
@@ -84,5 +84,5 @@
     <visual>
         <geometry>
-            <cylinder radius="0.05" length="0.04"/>
+            <cylinder radius="0.033" length="0.022"/>
         </geometry>
         <material name="blue"/>
@@ -90,8 +90,8 @@
     <collision>
         <geometry>
-            <cylinder radius="0.05" length="0.04"/>
+            <cylinder radius="0.033" length="0.022"/>
         </geometry>
     </collision>
-    <xacro:inertial_cylinder mass="0.1" length="0.04" radius="0.05">
+    <xacro:inertial_cylinder mass="0.1" radius="0.033" length="0.022">
         <origin xyz="0.0 0.0 0.0" rpy="0.0 0.0 0.0"/>
     </xacro:inertial_cylinder>
@@ -101,5 +101,5 @@
 </gazebo>
 <joint name="caster_wheel_joint" type="fixed">
-    <origin xyz="0.24 0.0 0.0" />
+    <origin xyz="0.1 0.0 0.0" />
     <parent link="chassis"/>
     <child link="caster_wheel"/>
@@ -108,5 +108,5 @@
     <visual>
         <geometry>
-            <sphere radius="0.05"/>
+            <sphere radius="0.033"/>
         </geometry>
         <material name="black"/>
@@ -114,8 +114,8 @@
     <collision>
         <geometry>
-            <sphere radius="0.05"/>
+            <sphere radius="0.033"/>
         </geometry>
     </collision>
-    <xacro:inertial_sphere mass="0.1" radius="0.05">
+    <xacro:inertial_sphere mass="0.1" radius="0.033">
         <origin xyz="0.0 0.0 0.0" rpy="0.0 0.0 0.0"/>
     </xacro:inertial_sphere>
